File: duct-turbo-fan-controller-v3/duct-turbo-fan-controller-v3.kicad_pcb (KiCad board)
At the start: 2 copper layers, 42.7 x 48.8 mm, 30 parts, among them J1 Screw_Terminal_01x04, J2 Conn_01x04, J3 USB_OTG, J4 AudioJack4, J7 Conn_01x04, Q1 MMBT3904, Q2 BSS84, SW1 SW_Push, SW2 SW_Push, U2 BME680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

Commit message: Connecting up the bme680/688 in pcb layout
Parts:
- moved R10 10.3 mm to (109.5, 83.3), turned to 0 degrees
- moved C6 9.80 mm to (112.6, 84.1), turned to 90 degrees
- moved R11 8.15 mm to (109.5, 84.8), turned to 0 degrees
- moved U2 0.11 mm to (110.5, 90.5)
Routing:
- net BME688_SCL: track 36.4 -> 57.6 mm, vias 0 -> 1
- net GND: track 24.4 -> 37.5 mm, vias 3 -> 4
- net BME688_SDA: track 51.4 -> 63.3 mm, vias 0 -> 1
- net Net-(U2-CSB): track 0.00 -> 11.4 mm, vias 0 -> 1
- net +3V3: track 136.3 -> 141.5 mm, vias 1 -> 2
- net Tacho: track 46.2 -> 44.5 mm
Other:
- outline, holes or cut-outs redrawn
- board text added: "DT/TB PWM Fan Controller v3.0"
- board text removed: "DT/TB PWM Fan Controller v2.5"
